File: pcb/lightlink/microcontroller_logic.kicad_sch (KiCad schematic)
At the start: 21 parts, among them J1 PIC Programming Header, J2 Wire Antenna, K1 Relay_SPST-NO, Q1 Q_NMOS_DGS, SW1 SW_DIP_x04, SW2 SW_MEC_5G_2LED, U1 PIC16F18126, U2 RFM69HCW

Commit message: Update PCB with several fixes
* Increase value of inrush limiting resistor
* Update locations of button/DIP switch
* Fix footprint for DIP switch
* Fix footprint for full bridge rectifier
* Change 1206 cap footprints to 0805
* Rotate main JST connector so that it doesn't impact the plug
Parts:
- SW1: footprint Package_DIP:DIP-8_W7.62mm -> switches_sps:DIP-8_SW_Horiz_Werth
Changed lines of the file:
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@@
       (effects (font (size 1.27 1.27)))
     )
-    (property "Footprint" "Package_DIP:DIP-8_W7.62mm" (at 233.68 142.24 0)
+    (property "Footprint" "switches_sps:DIP-8_SW_Horiz_Werth" (at 233.68 142.24 0)
       (effects (font (size 1.27 1.27)) hide)
     )

Commit message: Update PCB with couple fixes, cleanup code a bit
Parts:
- D3: value S1J-13-F -> ES1J-LTP
- D4: PN (none) -> HLMP1700; Part HLMP1700 -> (none)
- SW1: PN (none) -> 418217270904A
- SW2: PN (none) -> 228DD1S1AAFAMSC
Changed lines of the file:
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@@
+      (effects (font (size 1.27 1.27)) hide)
+    )
+    (property "PN" "228DD1S1AAFAMSC" (at 160.02 104.14 0)
       (effects (font (size 1.27 1.27)) hide)
     )
@@
       (effects (font (size 1.27 1.27)) (justify left))
     )
-    (property "Value" "S1J-13-F" (at 179.07 50.8 90)
+    (property "Value" "ES1J-LTP" (at 179.07 50.8 90)
       (effects (font (size 1.27 1.27)) (justify left))
     )
@@
       (effects (font (size 1.27 1.27)) hide)
     )
-    (property "Part" "HLMP1700" (at 41.91 102.87 90)
+    (property "PN" "HLMP1700" (at 41.91 102.87 90)
       (effects (font (size 1.27 1.27)) hide)
     )
@@
       (effects (font (size 1.27 1.27)) hide)
     )
+    (property "PN" "418217270904A" (at 233.68 142.24 0)
+      (effects (font (size 1.27 1.27)) hide)
+    )
