File: pcb/lightlink/power.kicad_sch (KiCad schematic)
At the start: 38 parts, among them J3 Conn_WallSocket, J4 Conn_01x01_Socket, J5 Conn_01x01_Socket, U3 LNK304G, U4 TPS56339DDC, U5 TLV3201

Commit message: Add released gerber files and fix board problem with reversed resistors
Parts:
- removed R15: 31.6k, Capacitor_SMD:C_0805_2012Metric_Pad1.18x1.45mm_HandSolder, symbol Device:R_US
- added R2: 31.6k, Capacitor_SMD:C_0805_2012Metric_Pad1.18x1.45mm_HandSolder, symbol Device:R_US
Connections:
- net +3.3V: now also R2.1; no longer R14.1
- net 3v3_FB: now also R14.1, R2.2; no longer R14.2
- net GND: now also R14.2

Commit message: Update PCB with several fixes
* Increase value of inrush limiting resistor
* Update locations of button/DIP switch
* Fix footprint for DIP switch
* Fix footprint for full bridge rectifier
* Change 1206 cap footprints to 0805
* Rotate main JST connector so that it doesn't impact the plug
Parts:
- C3, C5: footprint Capacitor_SMD:C_1206_3216Metric_Pad1.33x1.80mm_HandSolder -> Capacitor_SMD:C_0805_2012Metric_Pad1.18x1.45mm_HandSolder
- D2: part  (none) -> ES1J-LTP
- R9: value 10 - Fusible -> 20; Power (none) -> 3W
Connections:
- net LIVE_IN_FUSED: now also RV1.1
- net live_fbr_in: no longer RV1.1
Other:
- moved on the sheet: RV1
Changed lines of the file:
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@@
 (kicad_sch (version 20230121) (generator eeschema)
   (paper "A4")
+  (junction (at 59.69 34.29) (diameter 0) (color 0 0 0 0)
+  )
   (junction (at 114.3 107.95) (diameter 0) (color 0 0 0 0)
   )
@@
   (junction (at 186.69 107.95) (diameter 0) (color 0 0 0 0)
   )
-  (junction (at 81.28 34.29) (diameter 0) (color 0 0 0 0)
-  )
   (junction (at 201.93 59.69) (diameter 0) (color 0 0 0 0)
   )
@@
   (junction (at 200.66 107.95) (diameter 0) (color 0 0 0 0)
   )
-  (junction (at 59.69 34.29) (diameter 0) (color 0 0 0 0)
-  )
   (junction (at 36.83 34.29) (diameter 0) (color 0 0 0 0)
   )
@@
   (junction (at 160.02 59.69) (diameter 0) (color 0 0 0 0)
   )
-  (junction (at 81.28 49.53) (diameter 0) (color 0 0 0 0)
-  )
   (junction (at 50.8 49.53) (diameter 0) (color 0 0 0 0)
   )
@@
   (junction (at 165.1 59.69) (diameter 0) (color 0 0 0 0)
   )
+  (junction (at 66.04 34.29) (diameter 0) (color 0 0 0 0)
+  )
   (junction (at 133.35 107.95) (diameter 0) (color 0 0 0 0)
+  )
+  (junction (at 66.04 49.53) (diameter 0) (color 0 0 0 0)
   )
   (junction (at 201.93 41.91) (diameter 0) (color 0 0 0 0)
@@
     (stroke (width 0) (type default))
   )
+  (wire (pts (xy 66.04 49.53) (xy 104.14 49.53))
+    (stroke (width 0) (type default))
+  )
   (wire (pts (xy 160.02 59.69) (xy 160.02 62.23))
     (stroke (width 0) (type default))
@@
     (stroke (width 0) (type default))
   )
-  (wire (pts (xy 78.74 34.29) (xy 81.28 34.29))
-    (stroke (width 0) (type default))
-  )
   (wire (pts (xy 236.22 39.37) (xy 236.22 41.91))
     (stroke (width 0) (type default))
@@
     (stroke (width 0) (type default))
   )
+  (wire (pts (xy 86.36 34.29) (xy 104.14 34.29))
+    (stroke (width 0) (type default))
+  )
   (wire (pts (xy 248.92 110.49) (xy 254 110.49))
     (stroke (width 0) (type default))
   )
-  (wire (pts (xy 81.28 34.29) (xy 81.28 38.1))
+  (wire (pts (xy 66.04 34.29) (xy 66.04 36.83))
     (stroke (width 0) (type default))
   )
@@
     (stroke (width 0) (type default))
   )
+  (wire (pts (xy 66.04 34.29) (xy 78.74 34.29))
+    (stroke (width 0) (type default))
+  )
   (wire (pts (xy 165.1 54.61) (xy 165.1 59.69))
     (stroke (width 0) (type default))
@@
     (stroke (width 0) (type default))
   )
-  (wire (pts (xy 50.8 49.53) (xy 81.28 49.53))
-    (stroke (width 0) (type default))
-  )
   (wire (pts (xy 83.82 129.54) (xy 83.82 130.81))
     (stroke (width 0) (type default))
@@
     (stroke (width 0) (type default))
   )
-  (wire (pts (xy 81.28 49.53) (xy 104.14 49.53))
-    (stroke (width 0) (type default))
-  )
   (wire (pts (xy 26.67 39.37) (xy 50.8 39.37))
     (stroke (width 0) (type default))
@@
     (stroke (width 0) (type default))
   )
+  (wire (pts (xy 66.04 34.29) (xy 59.69 34.29))
+    (stroke (width 0) (type default))
+  )
   (wire (pts (xy 158.75 36.83) (xy 158.75 41.91))
     (stroke (width 0) (type default))
@@
     (stroke (width 0) (type default))
   )
-  (wire (pts (xy 81.28 34.29) (xy 104.14 34.29))
-    (stroke (width 0) (type default))
-  )
   (wire (pts (xy 248.92 120.65) (xy 248.92 124.46))
     (stroke (width 0) (type default))
@@
     (stroke (width 0) (type default))
   )
+  (wire (pts (xy 50.8 49.53) (xy 66.04 49.53))
+    (stroke (width 0) (type default))
+  )
   (wire (pts (xy 59.69 33.02) (xy 59.69 34.29))
     (stroke (width 0) (type default))
@@
     (stroke (width 0) (type default))
   )
-  (wire (pts (xy 59.69 34.29) (xy 71.12 34.29))
-    (stroke (width 0) (type default))
-  )
   (wire (pts (xy 147.32 129.54) (xy 133.35 129.54))
     (stroke (width 0) (type default))
   )
-  (wire (pts (xy 81.28 45.72) (xy 81.28 49.53))
+  (wire (pts (xy 66.04 44.45) (xy 66.04 49.53))
     (stroke (width 0) (type default))
   )
@@
       (effects (font (size 1.27 1.27)) hide)
     )
+    (property "part " "ES1J-LTP" (at 165.1 50.8 90)
+      (effects (font (size 1.27 1.27)) hide)
+    )
     (pin "1")
     (pin "2")
@@
     )
   )
-  (symbol (lib_id "Device:Varistor") (at 81.28 41.91 0) (unit 1)
-    (in_bom yes) (on_board yes) (dnp no) (fields_autoplaced)
-    (property "Reference" "RV1" (at 83.82 40.8333 0)
-      (effects (font (size 1.27 1.27)) (justify left))
-    )
-    (property "Value" "Varistor" (at 83.82 43.3733 0)
-      (effects (font (size 1.27 1.27)) (justify left))
-    )
-    (property "Footprint" "Varistor:RV_Disc_D7mm_W3.4mm_P5mm" (at 79.502 41.91 90)
-      (effects (font (size 1.27 1.27)) hide)
-    )
-    (property "Datasheet" "~" (at 81.28 41.91 0)
-      (effects (font (size 1.27 1.27)) hide)
-    )
-    (property "Sim.Name" "kicad_builtin_varistor" (at 81.28 41.91 0)
-      (effects (font (size 1.27 1.27)) hide)
-    )
-    (property "Sim.Device" "SUBCKT" (at 81.28 41.91 0)
-      (effects (font (size 1.27 1.27)) hide)
-    )
-    (property "Sim.Pins" "1=A 2=B" (at 81.28 41.91 0)
-      (effects (font (size 1.27 1.27)) hide)
-    )
-    (property "Sim.Params" "threshold=1k" (at 81.28 41.91 0)
-      (effects (font (size 1.27 1.27)) hide)
-    )
-    (property "Sim.Library" "${KICAD7_SYMBOL_DIR}/Simulation_SPICE.sp" (at 81.28 41.91 0)
+  (symbol (lib_id "Device:R_US") (at 82.55 34.29 90) (unit 1)
+    (in_bom yes) (on_board yes) (dnp no) (fields_autoplaced)
+    (property "Reference" "R9" (at 82.55 27.94 90)
+      (effects (font (size 1.27 1.27)))
+    )
+    (property "Value" "20" (at 82.55 30.48 90)
+      (effects (font (size 1.27 1.27)))
+    )
+    (property "Footprint" "Resistor_THT:R_Axial_DIN0207_L6.3mm_D2.5mm_P2.54mm_Vertical" (at 82.804 33.274 90)
+      (effects (font (size 1.27 1.27)) hide)
+    )
+    (property "Datasheet" "~" (at 82.55 34.29 0)
+      (effects (font (size 1.27 1.27)) hide)
+    )
+    (property "Power" "3W" (at 82.55 34.29 90)
+      (effects (font (size 1.27 1.27)) hide)
+    )
+    (pin "1")
+    (pin "2")
+    (instances
+      (project "lightlink"
+        (path "/7efd258b-cb88-4de5-af54-e5be8dd27051/28c50c9a-4c01-429d-8411-b6ccfebde60e"
+          (reference "R9") (unit 1)
+        )
+      )
+    )
+  )
+  (symbol (lib_id "Device:Varistor") (at 66.04 40.64 0) (unit 1)
+    (in_bom yes) (on_board yes) (dnp no) (fields_autoplaced)
+    (property "Reference" "RV1" (at 68.58 39.5633 0)
+      (effects (font (size 1.27 1.27)) (justify left))
+    )
+    (property "Value" "Varistor" (at 68.58 42.1033 0)
+      (effects (font (size 1.27 1.27)) (justify left))
+    )
+    (property "Footprint" "Varistor:RV_Disc_D7mm_W3.4mm_P5mm" (at 64.262 40.64 90)
+      (effects (font (size 1.27 1.27)) hide)
+    )
+    (property "Datasheet" "~" (at 66.04 40.64 0)
+      (effects (font (size 1.27 1.27)) hide)
+    )
+    (property "Sim.Name" "kicad_builtin_varistor" (at 66.04 40.64 0)
+      (effects (font (size 1.27 1.27)) hide)
+    )
+    (property "Sim.Device" "SUBCKT" (at 66.04 40.64 0)
+      (effects (font (size 1.27 1.27)) hide)
+    )
+    (property "Sim.Pins" "1=A 2=B" (at 66.04 40.64 0)
+      (effects (font (size 1.27 1.27)) hide)
+    )
+    (property "Sim.Params" "threshold=1k" (at 66.04 40.64 0)
+      (effects (font (size 1.27 1.27)) hide)
+    )
+    (property "Sim.Library" "${KICAD7_SYMBOL_DIR}/Simulation_SPICE.sp" (at 66.04 40.64 0)
       (effects (font (size 1.27 1.27)) hide)
     )
@@
       (effects (font (size 1.27 1.27)) (justify left))
     )
-    (property "Footprint" "Capacitor_SMD:C_1206_3216Metric_Pad1.33x1.80mm_HandSolder" (at 36.83 121.92 0)
+    (property "Footprint" "Capacitor_SMD:C_0805_2012Metric_Pad1.18x1.45mm_HandSolder" (at 36.83 121.92 0)
       (effects (font (size 1.27 1.27)) hide)
     )
@@
     )
   )
-  (symbol (lib_id "Device:R_US") (at 74.93 34.29 90) (unit 1)
-    (in_bom yes) (on_board yes) (dnp no) (fields_autoplaced)
-    (property "Reference" "R9" (at 74.93 27.94 90)
-      (effects (font (size 1.27 1.27)))
-    )
-    (property "Value" "10 - Fusible" (at 74.93 30.48 90)
-      (effects (font (size 1.27 1.27)))
-    )
-    (property "Footprint" "Resistor_THT:R_Axial_DIN0207_L6.3mm_D2.5mm_P2.54mm_Vertical" (at 75.184 33.274 90)
-      (effects (font (size 1.27 1.27)) hide)
-    )
-    (property "Datasheet" "~" (at 74.93 34.29 0)
-      (effects (font (size 1.27 1.27)) hide)
-    )
-    (pin "1")
-    (pin "2")
-    (instances
-      (project "lightlink"
-        (path "/7efd258b-cb88-4de5-af54-e5be8dd27051/28c50c9a-4c01-429d-8411-b6ccfebde60e"
-          (reference "R9") (unit 1)
-        )
-      )
-    )
-  )
   (symbol (lib_id "Device:C_Polarized_US") (at 185.42 31.75 0) (unit 1)
     (in_bom yes) (on_board yes) (dnp no) (fields_autoplaced)
@@
       (effects (font (size 1.27 1.27)) (justify left))
     )
-    (property "Footprint" "Capacitor_SMD:C_1206_3216Metric_Pad1.33x1.80mm_HandSolder" (at 185.42 31.75 0)
-      (effects (font (size 1.27 1.27)) hide)
-    )
+    (property "Footprint" "Capacitor_SMD:C_0805_2012Metric_Pad1.18x1.45mm_HandSolder" (at 185.42 31.75 0)
+      (effects (font (size 1.27 1.27)) hide)
+    )

Commit message: Update PCB with couple fixes, cleanup code a bit
Parts:
- D2: value ~ -> ES1J-LTP
- D3: value S1J-13-F -> ES1J-LTP
- D5: value 2.7V -> MM3Z2V7B 2.7V
- R9: value 20 -> 30; Power 3W -> 1W
Changed lines of the file:
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@@
   )
   (symbol (lib_id "Device:D") (at 165.1 50.8 270) (unit 1)
-    (in_bom yes) (on_board yes) (dnp no) (fields_autoplaced)
+    (in_bom yes) (on_board yes) (dnp no)
     (property "Reference" "D2" (at 167.64 50.8 90)
       (effects (font (size 1.27 1.27)) (justify left))
     )
-    (property "Value" "~" (at 167.64 52.07 90)
+    (property "Value" "ES1J-LTP" (at 167.64 53.34 90)
       (effects (font (size 1.27 1.27)) (justify left))
     )
@@
       (effects (font (size 1.27 1.27)))
     )
-    (property "Value" "TLV3201" (at 238.76 106.68 0)
+    (property "Value" "TLV3201" (at 238.76 115.57 0)
       (effects (font (size 1.27 1.27)))
     )
@@
       (effects (font (size 1.27 1.27)))
     )
-    (property "Value" "20" (at 82.55 30.48 90)
+    (property "Value" "30" (at 82.55 30.48 90)
       (effects (font (size 1.27 1.27)))
     )
@@
       (effects (font (size 1.27 1.27)) hide)
     )
-    (property "Power" "3W" (at 82.55 34.29 90)
+    (property "Power" "1W" (at 82.55 34.29 90)
       (effects (font (size 1.27 1.27)) hide)
     )
@@
       (effects (font (size 1.27 1.27)) (justify left))
     )
-    (property "Value" "2.7V" (at 180.34 116.84 90)
+    (property "Value" "MM3Z2V7B 2.7V" (at 176.53 118.11 90)
       (effects (font (size 1.27 1.27)) (justify left))
     )
@@
       (effects (font (size 1.27 1.27)) (justify left))
     )
-    (property "Value" "S1J-13-F" (at 204.47 34.29 90)
-      (effects (font (size 1.27 1.27)) (justify left))
-    )
+    (property "Value" "ES1J-LTP" (at 204.47 34.29 90)
+      (effects (font (size 1.27 1.27)) (justify left))
+    )
